Commit message: feat: copy urdf from previous attempt to make an auv

File: custom_robot_description/urdf/common_properties.xacro (robot description, xacro)
@@ -1,9 +1,18 @@
 <?xml version="1.0"?>
 <robot xmlns:xacro="http://www.ros.org/wiki/xacro">
-    <material name="blue">
-        <color rgba="0 0 0.5 1" />
-    </material>
     <material name="grey">
         <color rgba="0.5 0.5 0.5 1" />
     </material>
+    <material name="white">
+        <color rgba="1 1 1 1" />
+    </material>
+    <material name="orange">
+        <color rgba="1 0.3 0.1 1" />
+    </material>
+    <material name="blue">
+        <color rgba="0.2 0.2 1 1" />
+    </material>
+    <material name="black">
+        <color rgba="0 0 0 1" />
+    </material>
 </robot>

File: custom_robot_description/urdf/mobile_base.xacro (robot description, xacro)
@@ -1,62 +1,52 @@
 <?xml version="1.0"?>
 <robot xmlns:xacro="http://www.ros.org/wiki/xacro">
-    <xacro:property name="base_length" value="0.6" />
-    <xacro:property name="base_width" value="0.4" />
-    <xacro:property name="base_height" value="0.2" />
-    <xacro:property name="wheel_radius" value="0.1" />
-    <xacro:property name="wheel_length" value="0.05" />
-    <link name="base_footprint" />
-    <link name="base_link">
+    <xacro:property name="base_length" value="1.0" />
+    <xacro:property name="base_radius" value="0.4" />
+    <!-- <xacro:property name="base_width" value="0.4" /> -->
+    <!-- <xacro:property name="base_height" value="0.2" /> -->
+    <!-- <xacro:property name="wheel_radius" value="0.1" /> -->
+    <!-- <xacro:property name="wheel_length" value="0.05" /> -->
+    <!-- BASE LINK -->
+    <link name="base_link"></link>
+    <!-- CHASSIS LINK -->
+    <joint name="chassis_joint" type="fixed">
+        <parent link="base_link" />
+        <child link="chassis" />
+        <origin xyz="0 0 0" rpy="0 ${pi/2} 0" />
+    </joint>
+    <link name="chassis">
+        <visual>
+            <origin xyz="0 0 0" rpy="0 0 0" />
+            <geometry>
+                <cylinder radius="0.06" length="1.0" />
+            </geometry>
+            <material name="white" />
+        </visual>
+    </link>
+    <!-- PROPELLER LINK -->
+    <joint name="propeller_joint" type="continuous">
+        <parent link="base_link" />
+        <child link="propeller" />
+        <origin xyz="-0.51 0 0" rpy="0 ${pi/2} 0" />
+        <axis xyz="0 0 1" />
+    </joint>
+    <link name="propeller">
         <visual>
             <geometry>
-                <box size="${base_length} ${base_width} ${base_height}" />
+                <box size="0.2 0.02 0.01" />
             </geometry>
-            <origin xyz="0 0 ${base_height / 2.0}" rpy="0 0 0" />
-            <material name="blue" />
+            <material name="orange" />
         </visual>
+        <collision>
+            <geometry>
+                <box size="0.2 0.02 0.01" />
+            </geometry>
+        </collision>
+        <inertial>
+            <mass value="0.1" />
+            <inertia ixx="0.001" ixy="0" ixz="0"
+                iyy="0.001" iyz="0"
+                izz="0.001" />
+        </inertial>
     </link>
-    <xacro:macro name="wheel_link" params="prefix">
-        <link name="${prefix}_wheel_link">
-            <visual>
-                <geometry>
-                    <cylinder radius="${wheel_radius}" length="${wheel_length}" />
-                </geometry>
-                <origin xyz="0 0 0" rpy="${pi / 2.0} 0 0" />
-                <material name="grey" />
-            </visual>
-        </link>
-    </xacro:macro>
-    <xacro:wheel_link prefix="right" />
-    <xacro:wheel_link prefix="left" />
-    <link name="caster_wheel_link">
-        <visual>
-            <geometry>
-                <sphere radius="${wheel_radius / 2.0}" />
-            </geometry>
-            <origin xyz="0 0 0" rpy="0 0 0" />
-            <material name="grey" />
-        </visual>
-    </link>
-    <joint name="base_joint" type="fixed">
-        <parent link="base_footprint" />
-        <child link="base_link" />
-        <origin xyz="0 0 ${wheel_radius}" rpy="0 0 0"/>
-    </joint>
-    <joint name="base_right_wheel_joint" type="continuous">
-        <parent link="base_link" />
-        <child link="right_wheel_link" />
-        <origin xyz="${-base_length / 4.0} ${-(base_width + wheel_length) / 2.0} 0" rpy="0 0 0" />
-        <axis xyz="0 1 0" />
-    </joint>
-    <joint name="base_left_wheel_joint" type="continuous">
-        <parent link="base_link" />
-        <child link="left_wheel_link" />
-        <origin xyz="${-base_length / 4.0} ${(base_width + wheel_length) / 2.0} 0" rpy="0 0 0" />
-        <axis xyz="0 1 0" />
-    </joint>
-    <joint name="base_caster_wheel_joint" type="fixed">
-        <parent link="base_link" />
-        <child link="caster_wheel_link" />
-        <origin xyz="${base_length / 3.0} 0 ${-wheel_radius / 2.0}" rpy="0 0 0" />
-    </joint>
 </robot>

Commit message: feat: make it possible to launch custom robot in gazebo

File: custom_robot_description/urdf/common_properties.xacro (robot description, xacro)
@@ -16,3 +16,32 @@
         <color rgba="0 0 0 1" />
     </material>
+    <xacro:macro name="box_inertia" params="m x y z o_xyz o_rpy">
+        <inertial>
+            <mass value="${m}" />
+            <origin xyz="${o_xyz}" rpy="${o_rpy}" />
+            <inertia ixx="${(m/12) * (y*y + z*z)}" ixy="0" ixz="0"
+                iyy="${(m/12) * (x*x + z*z)}" iyz="0"
+                izz="${(m/12) * (x*x + y*y)}" />
+        </inertial>
+    </xacro:macro>
+    <xacro:macro name="sphere_inertia" params="m r o_xyz o_rpy">
+        <inertial>
+            <mass value="${m}" />
+            <origin xyz="${o_xyz}" rpy="${o_rpy}" />
+            <inertia ixx="${(2/5) * m * r * r}" ixy="0" ixz="0"
+                iyy="${(2/5) * m * r * r}" iyz="0"
+                izz="${(2/5) * m * r * r}" />
+        </inertial>
+    </xacro:macro>
+    <xacro:macro name="cylinder_inertia" params="m r l o_xyz o_rpy">
+        <inertial>
+            <mass value="${m}" />
+            <origin xyz="${o_xyz}" rpy="${o_rpy}" />
+            <inertia
+                ixx="${(m/12)*(3*r*r + l*l)}" ixy="0" ixz="0"
+                iyy="${(m/12)*(3*r*r + l*l)}" iyz="0"
+                izz="${(m/2)*(r*r)}"
+            />
+        </inertial>
+    </xacro:macro>
 </robot>

File: custom_robot_description/urdf/mobile_base.xacro (robot description, xacro)
@@ -2,9 +2,5 @@
 <robot xmlns:xacro="http://www.ros.org/wiki/xacro">
     <xacro:property name="base_length" value="1.0" />
-    <xacro:property name="base_radius" value="0.4" />
-    <!-- <xacro:property name="base_width" value="0.4" /> -->
-    <!-- <xacro:property name="base_height" value="0.2" /> -->
-    <!-- <xacro:property name="wheel_radius" value="0.1" /> -->
-    <!-- <xacro:property name="wheel_length" value="0.05" /> -->
+    <xacro:property name="base_radius" value="0.06" />
     <!-- BASE LINK -->
     <link name="base_link"></link>
@@ -19,8 +15,16 @@
             <origin xyz="0 0 0" rpy="0 0 0" />
             <geometry>
-                <cylinder radius="0.06" length="1.0" />
+                <cylinder radius="${base_radius}" length="${base_length}" />
             </geometry>
             <material name="white" />
         </visual>
+        <collision>
+            <geometry>
+                <cylinder radius="${base_radius}" length="${base_length}" />
+            </geometry>
+            <origin xyz="0 0 0" rpy="0 0 0" />
+        </collision>
+        <xacro:cylinder_inertia m="5.0" r="${base_radius}" l="${base_length}"
+            o_xyz="0 0 0" o_rpy="0 0 0" />
     </link>
     <!-- PROPELLER LINK -->
@@ -37,4 +41,5 @@
             </geometry>
             <material name="orange" />
+            <origin xyz="0 0 0" rpy="0 0 0" />
         </visual>
         <collision>
@@ -42,11 +47,8 @@
                 <box size="0.2 0.02 0.01" />
             </geometry>
+            <origin xyz="0 0 0" rpy="0 0 0" />
         </collision>
-        <inertial>
-            <mass value="0.1" />
-            <inertia ixx="0.001" ixy="0" ixz="0"
-                iyy="0.001" iyz="0"
-                izz="0.001" />
-        </inertial>
+        <xacro:box_inertia m="0.02" x="0.2" y="0.02" z="0.01"
+            o_xyz="0 0 0" o_rpy="0 0 0" />
     </link>
 </robot>
