Commit message: feat: clean up custom robot, to hopefully better fit its purpose

File: custom_robot_description/urdf/mobile_base.ros2_control.xacro (robot description, xacro)
@@ -6,13 +6,7 @@
             <param name="calculate_dynamics">true</param>
         </hardware>
-        <joint name="base_right_wheel_joint">
+        <joint name="propeller_joint">
             <command_interface name="velocity" />
             <state_interface name="position" />
-            <state_interface name="velocity" />
-        </joint>
-        <joint name="base_left_wheel_joint">
-            <command_interface name="velocity" />
-            <state_interface name="position" />
-            <state_interface name="velocity" />
         </joint>
     </ros2_control>

Commit message: fix: better structure of urdf to make things work properly-ish

File: custom_robot_description/urdf/mobile_base.ros2_control.xacro (robot description, xacro)
@@ -3,9 +3,9 @@
     <ros2_control name="MobileBaseHardwareInterface" type="system">
         <hardware>
-            <!-- <plugin>mock_components/GenericSystem</plugin>
-            <param name="calculate_dynamics">true</param> -->
-            <plugin>propeller_hardware/PropellerHardwareInterface</plugin>
+            <plugin>mock_components/GenericSystem</plugin>
+            <param name="calculate_dynamics">true</param>
+            <!-- <plugin>propeller_hardware/PropellerHardwareInterface</plugin>
             <param name="pigpiod_host">localhost</param>
-            <param name="pigpiod_port">8888</param>
+            <param name="pigpiod_port">8888</param> -->
         </hardware>
         <joint name="propeller_joint">

File: custom_robot_description/urdf/mobile_base.xacro (robot description, xacro)
@@ -3,15 +3,16 @@
     <xacro:property name="base_length" value="1.0" />
     <xacro:property name="base_radius" value="0.06" />
-    <!-- BASE LINK -->
-    <link name="base_link"></link>
-    <!-- CHASSIS LINK -->
-    <joint name="chassis_joint" type="fixed">
-        <parent link="base_link" />
-        <child link="chassis" />
-        <origin xyz="0 0 0" rpy="0 ${pi/2} 0" />
+    <xacro:property name="blade_full_length" value="0.1" />
+    <xacro:property name="blade_width" value="0.02" />
+    <xacro:property name="blade_height" value="0.01" />
+    <link name="base_footprint" />
+    <joint name="base_joint" type="fixed">
+        <parent link="base_footprint" />
+        <child link="base_link" />
+        <origin xyz="0 0 ${base_radius}" rpy="0 0 0" />
     </joint>
-    <link name="chassis">
+    <link name="base_link">
         <visual>
-            <origin xyz="0 0 0" rpy="0 0 0" />
+            <origin xyz="0 0 0" rpy="0 ${pi/2} 0" />
             <geometry>
                 <cylinder radius="${base_radius}" length="${base_length}" />
@@ -23,10 +24,9 @@
                 <cylinder radius="${base_radius}" length="${base_length}" />
             </geometry>
-            <origin xyz="0 0 0" rpy="0 0 0" />
+            <origin xyz="0 0 0" rpy="0 ${pi/2} 0" />
         </collision>
         <xacro:cylinder_inertia m="5.0" r="${base_radius}" l="${base_length}"
-            o_xyz="0 0 0" o_rpy="0 0 0" />
+            o_xyz="0 0 0" o_rpy="0 ${pi/2} 0" />
     </link>
-    <!-- PROPELLER LINK -->
     <joint name="propeller_joint" type="continuous">
         <parent link="base_link" />
@@ -38,5 +38,5 @@
         <visual>
             <geometry>
-                <box size="0.2 0.02 0.01" />
+                <box size="${blade_full_length} ${blade_width} ${blade_height}" />
             </geometry>
             <material name="orange" />
@@ -45,9 +45,9 @@
         <collision>
             <geometry>
-                <box size="0.2 0.02 0.01" />
+                <box size="${blade_full_length} ${blade_width} ${blade_height}" />
             </geometry>
             <origin xyz="0 0 0" rpy="0 0 0" />
         </collision>
-        <xacro:box_inertia m="0.02" x="0.2" y="0.02" z="0.01"
+        <xacro:box_inertia m="0.02" x="${blade_full_length}" y="${blade_width}" z="${blade_height}"
             o_xyz="0 0 0" o_rpy="0 0 0" />
     </link>
