Commit message: fix: use box as collision and 12 kg inertia which should work in gazebo

File: custom_robot_description/urdf/auv_base.xacro (robot description, xacro)
@@ -19,8 +19,10 @@
         <collision>
             <geometry>
-                <cylinder radius="${base_radius}" length="${base_length}" />
+                <box size="${2*base_radius} ${2*base_radius} ${base_length}" />
             </geometry>
             <origin xyz="0 0 0" rpy="0 ${pi/2} 0" />
         </collision>
+        <xacro:cylinder_inertia m="12.0" r="${base_radius}" l="${base_length}"
+            o_xyz="0 0 0" o_rpy="0 ${pi/2} 0" />
     </link>
 </robot>
