Commit message: refactor: remove obsolete commented code

File: custom_robot_description/urdf/auv_basic2.xacro (robot description, xacro)
@@ -1,17 +1,11 @@
 <?xml version="1.0"?>
 <robot name="auv" xmlns:xacro="http://www.ros.org/wiki/xacro">
-    <!-- Dummy root link -->
     <link name="base_link" />
-    <!-- Joint that rotates cylinder frame 90 degrees about Y -->
     <joint name="base_to_cylinder" type="fixed">
         <parent link="base_link" />
         <child link="cylinder_link" />
-        <!-- <origin xyz="0 0 0" rpy="0 1.57079632679 0" /> -->
-        <!-- lets not rotate it and see how it floats -->
         <origin xyz="0 0 0" rpy="0 0 0" />
     </joint>
-    <!-- Cylinder link -->
     <link name="cylinder_link">
-        <!-- Visual cylinder along Z axis (default) -->
         <visual>
             <origin xyz="0 0 0" rpy="0 ${pi/2} 0" />
@@ -23,24 +17,4 @@
             </material>
         </visual>
-        <!-- Collision box matching cylinder, no rotation -->
-        <!-- <collision>
-            <origin xyz="0 0 0" rpy="0 0 0" />
-            <geometry>
-                <box size="0.114 0.114 1.0" />
-            </geometry>
-        </collision> -->
-        <!-- Inertial with COM offset along local Z (radius) -->
-        <!-- <inertial>
-            <mass value="8.0" />
-            <origin xyz="0 0 0" rpy="0 0 0" />
-            <inertia
-                ixx="0.673165"
-                ixy="0"
-                ixz="0"
-                iyy="0.673165"
-                iyz="0"
-                izz="0.012996" />
-                </inertial> -->
-        <!-- partially stolen from tethys -->
         <collision>
             <geometry>
@@ -50,6 +24,4 @@
         </collision>
         <inertial>
-            <!-- <mass value="8.0" /> -->
-            <!-- <mass value="10.20186" /> -->
             <!-- this will make it neutral. use collision as volume -->
             <!-- <mass value="12.996" /> -->

File: custom_robot_description/urdf/auv_gazebo.xacro (robot description, xacro)
@@ -2,180 +2,10 @@
 <robot name="auv" xmlns:xacro="http://www.ros.org/wiki/xacro">
     <xacro:include filename="common_properties.xacro" />
-    <!-- <xacro:include filename="auv_base.xacro" /> -->
-    <!-- <xacro:include filename="auv_basic.xacro" /> -->
     <xacro:include filename="auv_basic2.xacro" />
-    <!-- <ros2_control name="Auv" type="system">
-        <hardware>
-            <plugin>mock_components/GenericSystem</plugin>
-        </hardware>
-    </ros2_control> -->
-    <!-- <gazebo>
-        <plugin filename="gz_ros2_control-system" name="gz_ros2_control::GazeboSimROS2ControlPlugin">
-            <parameters>$(find custom_robot_bringup)/config/auv_controllers.yaml</parameters>
-        </plugin>
-    </gazebo> -->
-    <!-- <gazebo reference="base_footprint">
-        <hejhej value="korv" />
-    </gazebo> -->
     <gazebo>
-        <!-- <plugin name='gz::sim::systems::Hydrodynamics' filename='gz-sim-hydrodynamics-system'>
-            <xDotU>-1.1</xDotU>
-            <yDotV>-11.3</yDotV>
-            <zDotW>-11.3</zDotW>
-            <kDotP>0</kDotP>
-            <mDotQ>0</mDotQ>
-            <nDotR>0</nDotR>
-            <xU>-5</xU>
-            <yV>-12</yV>
-            <zW>-10</zW>
-            <kP>0</kP>
-            <mQ>0</mQ>
-            <nR>0</nR>
-            <xUabsU>-4.6</xUabsU>
-            <yVabsV>-60</yVabsV>
-            <zWabsW>-60</zWabsW>
-            <kPabsP>-0.05</kPabsP>
-            <mQabsQ>-0.5</mQabsQ>
-            <nRabsR>-5</nRabsR>
-            <link_name>base_footprint</link_name>
-        </plugin> -->
         <plugin
             filename="gz-sim-hydrodynamics-system"
             name="gz::sim::systems::Hydrodynamics">
             <link_name>base_link</link_name>
-            <!-- works but floats wierdly -->
-            <!-- <xUabsU>0</xUabsU>
-            <xU>-30</xU>
-            <yVabsV>0</yVabsV>
-            <yV>-30</yV>
-            <zWabsW>0</zWabsW>
-            <zW>-30</zW>
-            <kPabsP>0</kPabsP>
-            <kP>-15</kP>
-            <mQabsQ>0</mQabsQ>
-            <mQ>-15</mQ>
-            <nRabsR>0</nRabsR>
-            <nR>-15</nR> -->
-            <!-- it's like if the Dot params make it crash? -->
-            <!-- <water_density>1000</water_density> -->
-            <!-- <xDotU>-4.876161</xDotU>
-            <yDotV>-126.324739</yDotV>
-            <zDotW>-126.324739</zDotW> -->
-            <!-- <kDotP>0</kDotP> -->
-            <!-- <mDotQ>-33.46</mDotQ>
-            <nDotR>-33.46</nDotR> -->
-            <!-- <xUabsU>-6.2282</xUabsU>
-            <xU>0</xU>
-            <yVabsV>-601.27</yVabsV>
-            <yV>0</yV>
-            <zWabsW>-601.27</zWabsW>
-            <zW>0</zW>
-            <kPabsP>-0.1916</kPabsP>
-            <kP>0</kP>
-            <mQabsQ>-632.698957</mQabsQ>
-            <mQ>0</mQ>
-            <nRabsR>-632.698957</nRabsR>
-            <nR>0</nR> -->
-            <!-- here are my values again, without Dot -->
-            <!-- <xDotU>-1.1</xDotU>
-            <yDotV>-5</yDotV>
-            <zDotW>-5</zDotW>
-            <kDotP>0</kDotP>
-            <mDotQ>0</mDotQ>
-            <nDotR>0</nDotR>
-            <xU>-5</xU>
-            <yV>-12</yV>
-            <zW>-10</zW>
-            <kP>0</kP>
-            <mQ>0</mQ>
-            <nR>0</nR>
-            <xUabsU>-4.6</xUabsU>
-            <yVabsV>-60</yVabsV>
-            <zWabsW>-60</zWabsW>
-            <kPabsP>-0.05</kPabsP>
-            <mQabsQ>-0.5</mQabsQ>
-            <nRabsR>-5</nRabsR> -->
-            <!-- <water_density>1000</water_density>
-            <xDotU>0</xDotU>
-            <yDotV>0</yDotV>
-            <zDotW>0</zDotW>
-            <kDotP>0</kDotP>
-            <mDotQ>0</mDotQ>
-            <nDotR>0</nDotR>
-            <xU>0</xU>
-            <yV>0</yV>
-            <zW>0</zW>
-            <kP>0</kP>
-            <mQ>0</mQ>
-            <nR>0</nR>
-            <xUabsU>-33.800000000000004</xUabsU>
-            <yVabsV>-54.26875</yVabsV>
-            <zWabsW>-73.37135</zWabsW>
-            <kPabsP>-4.0</kPabsP>
-            <mQabsQ>-4.0</mQabsQ>
-            <nRabsR>-4.0</nRabsR> -->
-            <!-- from chatty -->
-            <!-- <xDotU>-1.020703453</xDotU>
-            <yDotV>-5.207034532</yDotV>
-            <zDotW>-5.207034532</zDotW>
-            <kDotP>0.0</kDotP>
-            <mDotQ>0.0</mDotQ>
-            <nDotR>0.0</nDotR>
-            <xU>-5.0</xU>
-            <yV>-20.0</yV>
-            <zW>-20.0</zW>
-            <xUabsU>-1.020703453</xUabsU>
-            <yVabsV>-68.400000000</yVabsV>
-            <zWabsW>-68.400000000</zWabsW>
-            <default_current>0 0 0</default_current> -->
-            <!-- partially stolen from tethys -->
-            <!-- <xDotU>-1.876161</xDotU>
-            <yDotV>-8.324739</yDotV>
-            <zDotW>-8.324739</zDotW>
-            <kDotP>0</kDotP>
-            <mDotQ>-33.46</mDotQ>
-            <nDotR>-33.46</nDotR>
-            <xUabsU>-6.2282</xUabsU>
-            <xU>0</xU>
-            <yVabsV>-601.27</yVabsV>
-            <yV>0</yV>
-            <zWabsW>-601.27</zWabsW>
-            <zW>0</zW>
-            <kPabsP>-0.1916</kPabsP>
-            <kP>0</kP>
-            <mQabsQ>-632.698957</mQabsQ>
-            <mQ>0</mQ>
-            <nRabsR>-632.698957</nRabsR>
-            <nR>0</nR> -->
-            <!-- <xUabsU>0</xUabsU>
-            <xU>-30</xU>
-            <yVabsV>0</yVabsV>
-            <yV>-30</yV>
-            <zWabsW>0</zWabsW>
-            <zW>-30</zW>
-            <kPabsP>0</kPabsP>
-            <kP>-15</kP>
-            <mQabsQ>0</mQabsQ>
-            <mQ>-15</mQ>
-            <nRabsR>0</nRabsR>
-            <nR>-15</nR> -->
-            <!-- <xDotU>-1.1</xDotU>
-            <yDotV>-5</yDotV>
-            <zDotW>-5</zDotW>
-            <kDotP>0</kDotP>
-            <mDotQ>0</mDotQ>
-            <nDotR>0</nDotR>
-            <xU>-5</xU>
-            <yV>-12</yV>
-            <zW>-10</zW>
-            <kP>0</kP>
-            <mQ>0</mQ>
-            <nR>0</nR>
-            <xUabsU>-4.6</xUabsU>
-            <yVabsV>-60</yVabsV>
-            <zWabsW>-60</zWabsW>
-            <kPabsP>-0.05</kPabsP>
-            <mQabsQ>-0.5</mQabsQ>
-            <nRabsR>-5</nRabsR> -->
             <xDotU>-1.0</xDotU>
             <yDotV>-5</yDotV>
@@ -196,32 +26,5 @@
             <mQabsQ>-200</mQabsQ>
             <nRabsR>-100</nRabsR>
-            <!-- <xDotU>-1.0</xDotU>
-            <yDotV>0</yDotV>
-            <zDotW>0</zDotW>
-            <kDotP>0</kDotP>
-            <mDotQ>0</mDotQ>
-            <nDotR>0</nDotR>
-            <xU>0</xU>
-            <yV>0</yV>
-            <zW>0</zW>
-            <kP>0</kP>
-            <mQ>0</mQ>
-            <nR>0</nR>
-            <xUabsU>0</xUabsU>
-            <yVabsV>0</yVabsV>
-            <zWabsW>0</zWabsW>
-            <kPabsP>0</kPabsP>
-            <mQabsQ>0</mQabsQ>
-            <nRabsR>0</nRabsR> -->
         </plugin>
-        <!-- <plugin name="gz::sim::systems::Hydrodynamics"
-        filename="gz-waves1-hydrodynamics-system">
-            <enable>auv::base_link</enable>
-            <hydrodynamics>
-                <damping_on>1</damping_on>
-                <viscous_drag_on>1</viscous_drag_on>
-                <pressure_drag_on>1</pressure_drag_on>
-            </hydrodynamics>
-        </plugin> -->
     </gazebo>
 </robot>

Commit message: feat: working setup with making auv move with ros commands

File: custom_robot_description/urdf/auv_basic2.xacro (robot description, xacro)
@@ -1,4 +1,9 @@
 <?xml version="1.0"?>
 <robot name="auv" xmlns:xacro="http://www.ros.org/wiki/xacro">
+    <xacro:property name="base_length" value="1.0" />
+    <xacro:property name="base_radius" value="0.057" />
+    <xacro:property name="thruster_radius" value="0.045" />
+    <xacro:property name="thruster_thickness" value="0.01" />
+    <xacro:property name="thruster_offset" value="0.01" />
     <link name="base_link" />
     <joint name="base_to_cylinder" type="fixed">
@@ -11,5 +16,5 @@
             <origin xyz="0 0 0" rpy="0 ${pi/2} 0" />
             <geometry>
-                <cylinder length="1.0" radius="0.057" />
+                <cylinder length="${base_length}" radius="${base_radius}" />
             </geometry>
             <material name="color1">
@@ -19,5 +24,5 @@
         <collision>
             <geometry>
-                <box size="1 0.114 0.114" />
+                <box size="${base_length} ${base_radius*2} ${base_radius*2}" />
             </geometry>
             <origin xyz="0 0 0" rpy="0 0 0" />
@@ -38,3 +43,40 @@
         </inertial>
     </link>
+    <link name="thruster_link">
+        <visual>
+            <origin xyz="0 0 0" rpy="0 0 0" />
+            <geometry>
+                <!-- <cylinder length="${thruster_thickness}" radius="${thruster_radius}" /> -->
+                <box size="${thruster_thickness} ${thruster_radius*2} ${thruster_thickness}" />
+            </geometry>
+            <material name="blueish">
+                <color rgba="0.3 0.3 0.9 1" />
+            </material>
+        </visual>
+        <collision>
+            <origin xyz="0 0 0" rpy="0 0 0" />
+            <geometry>
+                <!-- <cylinder length="${thruster_thickness}" radius="${thruster_radius}" /> -->
+                <!-- <box size="${thruster_thickness} ${thruster_radius*2} ${thruster_radius*2}" /> -->
+                <sphere radius="0.005" />
+            </geometry>
+        </collision>
+        <xacro:sphere_inertia m="0.001" r="0.005"
+            o_xyz="0 0 0" o_rpy="0 0 0" />
+        <!-- <inertial>
+            <origin xyz="0 0 0" rpy="0 0 0" />
+            <mass value="0.001" />
+            <inertia ixx="1e-4" ixy="0" ixz="0" iyy="1e-4" iyz="0" izz="1e-4" />
+        </inertial> -->
+    </link>
+    <joint name="cylinder_thruster_joint" type="continuous">
+        <parent link="cylinder_link" />
+        <child link="thruster_link" />
+        <origin xyz="-${base_length/2 + thruster_thickness/2 + thruster_offset} 0 0" rpy="0 0 0" />
+        <axis xyz="1 0 0" />
+        <limit lower="0" upper="100" effort="100" velocity="100" />
+        <!-- <axis xyz="0 0 1" /> -->
+        <!-- <limit lower="0" upper="${pi/2}" effort="100" velocity="100" />
+        <dynamics friction="0.05" damping="0.1" /> -->
+    </joint>
 </robot>

File: custom_robot_description/urdf/auv_gazebo.xacro (robot description, xacro)
@@ -28,3 +28,61 @@
         </plugin>
     </gazebo>
+    <ros2_control name="Auv" type="system">
+        <hardware>
+            <plugin>gz_ros2_control/GazeboSimSystem</plugin>
+            <!-- <plugin>mock_components/GenericSystem</plugin> -->
+        </hardware>
+        <joint name="cylinder_thruster_joint">
+            <command_interface name="velocity" />
+            <state_interface name="position" />
+            <state_interface name="velocity" />
+        </joint>
+    </ros2_control>
+    <gazebo>
+        <plugin filename="gz_ros2_control-system" name="gz_ros2_control::GazeboSimROS2ControlPlugin">
+            <parameters>$(find custom_robot_bringup)/config/auv_controllers.yaml</parameters>
+        </plugin>
+        <!-- </gazebo> -->
+        <!-- <plugin
+      filename="gz-sim-thruster-system"
+      name="gz::sim::systems::Thruster"> -->
+        <!-- <joint_name>${namespace}/${name}_engine_propeller_joint</joint_name>
+      <thrust_coefficient>0.004422</thrust_coefficient>
+      <fluid_density>1000</fluid_density>
+      <propeller_diameter>0.2</propeller_diameter>
+      <velocity_control>true</velocity_control>
+      <max_thrust_cmd>${((x_u + x_uu * max_velocity_mps) * max_velocity_mps)/ 2}</max_thrust_cmd>
+      <namespace>${namespace}</namespace>
+      <topic>thrusters/${name}/thrust</topic>
+      <name>${name}</name>  -->
+        <!-- gz::sim::systems::Thruster -->
+        <!-- <gazebo> -->
+        <plugin
+            filename="gz-sim-thruster-system"
+            name="gz::sim::systems::Thruster"
+        >
+            <!-- <plugin name="thruster" filename="libgz-sim-systems-thruster.so"> -->
+            <joint_name>cylinder_thruster_joint</joint_name>      <!-- the joint you created in your URDF -->
+            <topic>thruster0/cmd_thrust</topic>           <!-- plugin will listen on this gz topic -->
+            <use_angvel_cmd>false</use_angvel_cmd>        <!-- we send thrust (N) -->
+            <velocity_control>false</velocity_control>    <!-- let plugin apply wrenches directly -->
+            <thrust_coefficient>1.0</thrust_coefficient>
+            <fluid_density>1000</fluid_density>
+            <propeller_diameter>0.2</propeller_diameter>
+            <velocity_control>true</velocity_control>
+            <max_thrust_cmd>50</max_thrust_cmd>
+            <name>auv</name>
+        </plugin>
+    </gazebo>
+    <!-- <gazebo>
+        <plugin
+            filename="gz-sim-joint-state-publisher-system"
+            name="gz::sim::systems::JointStatePublisher"
+        >
+            <joint_name>base_left_wheel_joint</joint_name>
+            <joint_name>base_right_wheel_joint</joint_name>
+            <joint_name>arm_base_forearm_joint</joint_name>
+            <joint_name>forearm_hand_joint</joint_name>
+        </plugin>
+    </gazebo> -->
 </robot>

Commit message: feat: make propeller spin (at least in rviz)

File: custom_robot_description/urdf/auv_basic2.xacro (robot description, xacro)
@@ -75,5 +75,4 @@
         <origin xyz="-${base_length/2 + thruster_thickness/2 + thruster_offset} 0 0" rpy="0 0 0" />
         <axis xyz="1 0 0" />
-        <limit lower="0" upper="100" effort="100" velocity="100" />
         <!-- <axis xyz="0 0 1" /> -->
         <!-- <limit lower="0" upper="${pi/2}" effort="100" velocity="100" />
