Commit message: feat: join hull and thruster together, and make it possible to run with controllers in gazebo

File: custom_robot_description/urdf/auv.urdf.xacro (robot description, xacro)
@@ -2,5 +2,10 @@
 <robot name="auv" xmlns:xacro="http://www.ros.org/wiki/xacro">
     <xacro:include filename="common_properties.xacro" />
-    <!-- <xacro:include filename="auv_basic2.xacro" /> -->
-    <xacro:include filename="steerable_propeller.xacro" />
+    <xacro:include filename="auv_basic2.xacro" />
+    <xacro:include filename="auv_thrust.xacro" />
+    <joint name="base_rudder_base_joint" type="fixed">
+        <parent link="cylinder_link" />
+        <child link="rudder_base" />
+        <origin xyz="-${base_length/2} 0 0" rpy="0 0 ${pi}" />
+    </joint>
 </robot>

File: custom_robot_description/urdf/auv_basic2.xacro (robot description, xacro)
@@ -31,5 +31,6 @@
             <!-- this will make it neutral. use collision as volume -->
             <!-- <mass value="12.996" /> -->
-            <mass value="10.996" />
+            <mass value="12" />
+            <!-- <mass value="10.996" /> -->
             <inertia
                 ixx="0.018"
@@ -43,39 +44,3 @@
         </inertial>
     </link>
-    <link name="thruster_link">
-        <visual>
-            <origin xyz="0 0 0" rpy="0 0 0" />
-            <geometry>
-                <!-- <cylinder length="${thruster_thickness}" radius="${thruster_radius}" /> -->
-                <box size="${thruster_thickness} ${thruster_radius*2} ${thruster_thickness}" />
-            </geometry>
-            <material name="blueish">
-                <color rgba="0.3 0.3 0.9 1" />
-            </material>
-        </visual>
-        <collision>
-            <origin xyz="0 0 0" rpy="0 0 0" />
-            <geometry>
-                <!-- <cylinder length="${thruster_thickness}" radius="${thruster_radius}" /> -->
-                <!-- <box size="${thruster_thickness} ${thruster_radius*2} ${thruster_radius*2}" /> -->
-                <sphere radius="0.005" />
-            </geometry>
-        </collision>
-        <xacro:sphere_inertia m="0.001" r="0.005"
-            o_xyz="0 0 0" o_rpy="0 0 0" />
-        <!-- <inertial>
-            <origin xyz="0 0 0" rpy="0 0 0" />
-            <mass value="0.001" />
-            <inertia ixx="1e-4" ixy="0" ixz="0" iyy="1e-4" iyz="0" izz="1e-4" />
-        </inertial> -->
-    </link>
-    <joint name="cylinder_thruster_joint" type="continuous">
-        <parent link="cylinder_link" />
-        <child link="thruster_link" />
-        <origin xyz="-${base_length/2 + thruster_thickness/2 + thruster_offset} 0 0" rpy="0 0 0" />
-        <axis xyz="1 0 0" />
-        <!-- <axis xyz="0 0 1" /> -->
-        <!-- <limit lower="0" upper="${pi/2}" effort="100" velocity="100" />
-        <dynamics friction="0.05" damping="0.1" /> -->
-    </joint>
 </robot>

File: custom_robot_description/urdf/auv_gazebo.xacro (robot description, xacro)
@@ -1,6 +1,5 @@
 <?xml version="1.0"?>
 <robot name="auv" xmlns:xacro="http://www.ros.org/wiki/xacro">
-    <xacro:include filename="common_properties.xacro" />
-    <xacro:include filename="auv_basic2.xacro" />
+    <xacro:include filename="auv.urdf.xacro" />
     <gazebo>
         <plugin
@@ -37,4 +36,12 @@
             <state_interface name="position" />
             <state_interface name="velocity" />
+        </joint>
+        <joint name="yaw_joint">
+            <command_interface name="position" />
+            <state_interface name="position" />
+        </joint>
+        <joint name="pitch_joint">
+            <command_interface name="position" />
+            <state_interface name="position" />
         </joint>
     </ros2_control>

File: custom_robot_description/urdf/auv_ros2_control.xacro (robot description, xacro)
@@ -1,6 +1,5 @@
 <?xml version="1.0"?>
 <robot name="auv" xmlns:xacro="http://www.ros.org/wiki/xacro">
-    <xacro:include filename="common_properties.xacro" />
-    <xacro:include filename="auv_basic2.xacro" />
+    <xacro:include filename="auv.urdf.xacro" />
     <ros2_control name="Auv" type="system">
         <hardware>
@@ -13,4 +12,12 @@
             <state_interface name="velocity" />
         </joint>
+        <joint name="yaw_joint">
+            <command_interface name="position" />
+            <state_interface name="position" />
+        </joint>
+        <joint name="pitch_joint">
+            <command_interface name="position" />
+            <state_interface name="position" />
+        </joint>
     </ros2_control>
 </robot>

File: custom_robot_description/urdf/auv_thrust.xacro (robot description, xacro)
@@ -1,15 +1,17 @@
 <?xml version="1.0"?>
 <robot xmlns:xacro="http://www.ros.org/wiki/xacro">
-    <xacro:property name="rudder_base_side" value="0.05" />
-    <xacro:property name="rudder_base_thickness" value="0.005" />
-    <xacro:property name="axis_length" value="0.05" />
-    <xacro:property name="axis_radius" value="0.005" />
+    <xacro:property name="rudder_base_radius" value="0.005" />
+    <xacro:property name="axis_length" value="0.02" />
+    <xacro:property name="axis_radius" value="0.001" />
     <xacro:property name="yaw_limit_rad" value="0.785" />
     <xacro:property name="pitch_limit_rad" value="0.5" />
+    <xacro:property name="thruster_radius" value="0.03" />
+    <xacro:property name="thruster_thickness" value="0.002" />
+    <xacro:property name="thruster_blade_width" value="0.01" />
     <link name="rudder_base">
         <visual>
             <origin xyz="0 0 0" rpy="0 0 0" />
             <geometry>
-                <box size="${rudder_base_thickness} ${rudder_base_side} ${rudder_base_side}" />
+                <sphere radius="${rudder_base_radius}" />
             </geometry>
             <material name="yellowish1">
@@ -20,12 +22,10 @@
             <origin xyz="0 0 0" rpy="0 0 0" />
             <geometry>
-                <box size="${rudder_base_thickness} ${rudder_base_side} ${rudder_base_side}" />
+                <sphere radius="${rudder_base_radius}" />
             </geometry>
         </collision>
-        <xacro:box_inertia
+        <xacro:sphere_inertia
             m="0.001"
-            x="${rudder_base_thickness}"
-            y="${rudder_base_side}"
-            z="${rudder_base_side}"
+            r="${rudder_base_radius}"
             o_xyz="0 0 0"
             o_rpy="0 0 0"
@@ -59,9 +59,15 @@
         <parent link="rudder_base" />
         <child link="rod_intermediate_link" />
-        <origin xyz="${rudder_base_thickness/2} 0 0" rpy="0 0 0" />
+        <origin xyz="${rudder_base_radius} 0 0" rpy="0 0 0" />
         <axis xyz="0 0 1" />
         <limit lower="-${yaw_limit_rad}" upper="${yaw_limit_rad}" effort="100" velocity="100" />
     </joint>
-    <link name="rod_intermediate_link"></link>
+    <link name="rod_intermediate_link">
+        <inertial>
+            <mass value="0.0001" />
+            <inertia ixx="0.0001" ixy="0.0" ixz="0.0" iyy="0.0001" iyz="0.0" izz="0.0001" />
+            <origin xyz="0 0 0" rpy="0 0 0" />
+        </inertial>
+    </link>
     <joint name="pitch_joint" type="revolute">
         <parent link="rod_intermediate_link" />
@@ -70,3 +76,28 @@
         <limit lower="-${pitch_limit_rad}" upper="${pitch_limit_rad}" effort="100" velocity="100" />
     </joint>
+    <link name="thruster_link">
+        <visual>
+            <origin xyz="0 0 0" rpy="0 0 0" />
+            <geometry>
+                <box size="${thruster_thickness} ${thruster_radius*2} ${thruster_blade_width}" />
+            </geometry>
+            <material name="blueish">
+                <color rgba="0.3 0.3 0.9 1" />
+            </material>
+        </visual>
+        <collision>
+            <origin xyz="0 0 0" rpy="0 0 0" />
+            <geometry>
+                <sphere radius="0.005" />
+            </geometry>
+        </collision>
+        <xacro:sphere_inertia m="0.001" r="0.005"
+            o_xyz="0 0 0" o_rpy="0 0 0" />
+    </link>
+    <joint name="cylinder_thruster_joint" type="continuous">
+        <parent link="rod_link" />
+        <child link="thruster_link" />
+        <origin xyz="${axis_length + thruster_thickness/2} 0 0" rpy="0 0 0" />
+        <axis xyz="-1 0 0" />
+    </joint>
 </robot>
